File: Zegar na oscyloskop.sch (KiCad schematic (older format))
At the start: 23 parts

Commit message: Finished
Parts:
- removed C?: 105, symbol Device:C
- removed C?: 100n, symbol Device:C
- removed R?: 10k, symbol Device:R
- removed R?: 3.3k, symbol Device:R
- removed RV?: 1k, symbol Device:R_POT
- removed U?: XL4015, symbol hello_there:XL4015
- added C15, C2: 10u, Capacitor_THT:CP_Radial_D4.0mm_P1.50mm, symbol Device:CP
- added C16, C4, C7, C8: 100n, Capacitor_THT:C_Rect_L7.0mm_W3.5mm_P5.00mm, symbol Device:C
- added D2, D3, D4, D5: LED, LED_THT:LED_D5.0mm_Clear, symbol Device:LED
- added J2: USB_B, Connector_USB:USB_B_OST_USB-B1HSxx_Horizontal, symbol Connector:USB_B
- added J3: PROG, Connector_PinHeader_2.54mm:PinHeader_2x05_P2.54mm_Vertical, symbol Connector_Generic:Conn_02x05_Odd_Even
- added J4, J5: BNC, Connector_Coaxial:BNC_Amphenol_B6252HB-NPP3G-50_Horizontal, symbol Connector:Conn_Coaxial
- added J6, J7: BNC, Connector_Wire:SolderWirePad_1x02_P5.08mm_Drill1.5mm, symbol Connector:Conn_Coaxial
- added R1, R13, R14, R15, R16: 10k, Resistor_THT:R_Axial_DIN0207_L6.3mm_D2.5mm_P10.16mm_Horizontal, symbol Device:R
- added R11, R12, R2, R3, R4, R5, R6, R7, R8, R9: 1k, Resistor_THT:R_Axial_DIN0207_L6.3mm_D2.5mm_P10.16mm_Horizontal, symbol Device:R
- added SW1: H, Button_Switch_THT:SW_PUSH_6mm_H5mm, symbol Switch:SW_Push
- added SW2: M, Button_Switch_THT:SW_PUSH_6mm_H5mm, symbol Switch:SW_Push
- added SW3: S, Button_Switch_THT:SW_PUSH_6mm_H5mm, symbol Switch:SW_Push
- added SW4: L, Button_Switch_THT:SW_PUSH_6mm_H5mm, symbol Switch:SW_Push
- added U2: LM2596T-5, Package_TO_SOT_THT:TO-220-5_P3.4x3.7mm_StaggerOdd_Lead3.8mm_Vertical, symbol Regulator_Switching:LM2596T-5
- added U3: FT232RL, Package_SO:SSOP-28_5.3x10.2mm_P0.65mm, symbol Interface_USB:FT232RL
- C1, C11, C13: renamed from C?; footprint (none) -> Capacitor_THT:C_Rect_L7.0mm_W3.5mm_P5.00mm
- C10, C6: renamed from C?; footprint (none) -> Capacitor_THT:CP_Radial_D4.0mm_P1.50mm
- C12, C5: renamed from C?; value 105 -> 100n; footprint (none) -> Capacitor_THT:C_Rect_L7.0mm_W3.5mm_P5.00mm
- C3: renamed from C?; value 220u -> 680u; footprint (none) -> Capacitor_THT:CP_Radial_D10.0mm_P5.00mm
- C9: renamed from C?; value 330u -> 220u; footprint (none) -> Capacitor_THT:CP_Radial_D10.0mm_P5.00mm
- D1: renamed from D?; value 1N5818 -> 1N5824; footprint (none) -> Diode_THT:D_DO-201AD_P15.24mm_Horizontal
- J1: renamed from J?; footprint (none) -> Connector_Wire:SolderWirePad_1x02_P5.08mm_Drill1.5mm
- L1: renamed from L?; value 47u -> 33u; footprint (none) -> Inductor_SMD:L_12x12mm_H6mm
- L2: renamed from L?; footprint (none) -> Inductor_THT:L_Axial_L6.6mm_D2.7mm_P10.16mm_Horizontal_Vishay_IM-2
- R10: renamed from R?; footprint (none) -> Resistor_THT:R_Axial_DIN0207_L6.3mm_D2.5mm_P10.16mm_Horizontal
- U4: renamed from U?; footprint (none) -> Package_DIP:DIP-24_W7.62mm_Socket; symbol hello_there:MAX505 -> Zegar-na-oscyloskop-rescue:MAX505-hello_there
- U5: renamed from U?; footprint Package_DIP:DIP-28_W7.62mm -> Package_DIP:DIP-28_W7.62mm_Socket; symbol MCU_Microchip_ATmega:ATmega8A-PU -> Zegar-na-oscyloskop-rescue:ATmega8A-PU-MCU_Microchip_ATmega
- gave numbers to parts that had none: 1
Connections:
- net +5V: now also C15.1, C16.1, C2.1, C4.1, D2.2 (A), D3.2 (A), J3.2 (Pin_2), R1.1, U2.4 (FB), U3.20 (VCC), U3.4 (VCCIO)
- net A0: now also U5.14 (PB0)
- net A1: now also U5.15 (PB1)
- net D0: now also U5.17 (PB3), J3.1 (Pin_1)
- net D1: now also U5.18 (PB4), J3.9 (Pin_9)
- net D2: now also U5.19 (PB5), J3.7 (Pin_7)
- net D3: now also U5.23 (PC0)
- net D4: now also U5.24 (PC1)
- net D5: now also U5.25 (PC2)
- net D6: now also U5.26 (PC3)
- net D7: now also U5.27 (PC4)
- net GND: now also C15.2, C16.2, C2.2, C4.2, C7.2, D4.1 (K), D5.1 (K), J2.4 (GND), J2.5 (Shield), J3.10 (Pin_10), J3.4 (Pin_4), J3.6 (Pin_6), J3.8 (Pin_8), J4.2 (Ext), J5.2 (Ext), J6.2 (Ext), J7.2 (Ext), SW1.2, SW2.2, SW3.2, SW4.2, U2.3 (GND), U2.5 (~ON~/OFF), U3.18 (GND), U3.21 (GND), U3.25 (AGND), U3.26 (TEST), U3.7 (GND)
- net LDAC: now also U5.28 (PC5)
- net OUT_A: now also R6.2
- net OUT_B: now also R7.2
- net OUT_C: now also R8.2
- net OUT_D: now also R9.2
- net WR: now also U5.16 (PB2)
- net at C3.1, C5.1, J1.1 (Pin_1): now also U2.1 (VIN)
- net at D1.1 (K), L1.1: now also U2.2 (OUT)
- net RST: now reaches R10.2, U5.1 (PC6/~RESET)
- net RST: now also C8.1, J3.5 (Pin_5)
- net BTN_M: now reaches U5.10 (PB7/XTAL2)
- net BTN_M: now also R14.1
- net BTN_S: now reaches U5.11 (PD5)
- net BTN_S: now also R15.1
- net BTN_L: now reaches U5.12 (PD6)
- net BTN_L: now also R16.1
- net UC_RXD: now reaches U5.2 (PD0)
- net UC_RXD: now also R2.1
- net UC_TXD: now reaches U5.3 (PD1)
- net UC_TXD: now also R5.1
- net LED_1: now reaches U5.4 (PD2)
- net LED_1: now also R11.2
- net LED_2: now reaches U5.5 (PD3)
- net LED_2: now also R12.2
- net BTN_H: now reaches U5.9 (PB6/XTAL1)
- net BTN_H: now also R13.1
- new net: D4.2 (A), R11.1
- new net: D5.2 (A), R12.1
- new net: R13.2, SW1.1
- new net: R14.2, SW2.1
- new net: R15.2, SW3.1
- new net: R16.2, SW4.1
- new net: R2.2, U3.1 (TXD)
- new net: C7.1, U3.17 (3V3OUT)
- new net: R1.2, U3.19 (~RESET~)
- new net: C8.2, U3.2 (DTR)
- new net: R3.2, U3.22 (CBUS1)
- new net: R4.2, U3.23 (CBUS0)
- new net: R5.2, U3.5 (RXD)
- new net: D3.1 (K), R3.1
- new net: D2.1 (K), R4.1
- new net: J4.1 (In), R6.1
- new net: J5.1 (In), R7.1
- new net: J6.1 (In), R8.1
- new net: J7.1 (In), R9.1
- new net D+: J2.3 (D+), U3.15 (USBD+)
- new net D-: J2.2 (D-), U3.16 (USBD-)
- no-connect marks 0 -> 15
Other:
- note added: "BNC"
- note added: "CPU"
- note added: "CPU I/O"
- note added: "Prog"
- note added: "USB"
- moved on the sheet: C1, C10, C11, C12, C13, C3, C5, C6, C9, D1, J1, L1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
